Commit message: added namespace to all sensors

File: urdf/econ/see3cam.urdf.xacro (robot description, xacro)
@@ -7,7 +7,7 @@
         <xacro:insert_block name="origin" />
         <parent link="${parent}"/>
-        <child link="${name}_link" />
+        <child link="${namespace}/${name}_link" />
     </joint>
-    <link name="${name}_link">
+    <link name="${namespace}/${name}_link">
         <inertial>
             <mass value="0.05" />
@@ -32,15 +32,15 @@
         </collision>
     </link>
-    <gazebo reference="${name}_link">
+    <gazebo reference="${namespace}/${name}_link">
         <material>Gazebo/FlatBlack</material>
     </gazebo>
     <joint name="${name}_optical_frame_joint" type="fixed">
         <origin xyz="0.0 0 0" rpy="0 0 0"/>
-        <parent link="${name}_link"/>
-        <child link="${name}_optical_link"/>
+        <parent link="${namespace}/${name}_link"/>
+        <child link="${namespace}/${name}_optical_link"/>
     </joint>
-    <link name="${name}_optical_link"/>
+    <link name="${namespace}/${name}_optical_link"/>
     <!-- extension -->
-    <xacro:gazebo_camera name="${name}_image" reference="${name}_optical_link" hz="${hz}" h_fov="${h_fov}" width="1920" height="1080" format="${format}" frame_id="${name}_link"/>
+    <xacro:gazebo_camera name="${name}_image" reference="${name}_optical_link" hz="${hz}" h_fov="${h_fov}" width="1920" height="1080" format="${format}" frame_id="${namespace}/${name}_link"/>
     </xacro:macro>
 </robot>

File: urdf/flir/firefly.urdf.xacro (robot description, xacro)
@@ -7,7 +7,7 @@
         <xacro:insert_block name="origin" />
         <parent link="${parent}"/>
-        <child link="${name}_link" />
+        <child link="${namespace}/${name}_link" />
     </joint>
-    <link name="${name}_link">
+    <link name="${namespace}/${name}_link">
         <inertial>
             <mass value="0.05" />
@@ -29,15 +29,15 @@
         </collision>
     </link>
-    <gazebo reference="${name}_link">
+    <gazebo reference="${namespace}/${name}_link">
         <material>Gazebo/FlatBlack</material>
     </gazebo>
     <joint name="${name}_optical_frame_joint" type="fixed">
         <origin xyz="0.0 0 0" rpy="0 0 0"/>
-        <parent link="${name}_link"/>
+        <parent link="${namespace}/${name}_link"/>
         <child link="${name}_optical_link"/>
     </joint>
     <link name="${name}_optical_link"/>
     <!-- extension -->
-    <xacro:gazebo_camera name="${name}_image" reference="${name}_optical_link" hz="${hz}" h_fov="${h_fov}" width="1440" height="1080" format="${format}" frame_id="${name}_link"/>
+    <xacro:gazebo_camera name="${name}_image" reference="${name}_optical_link" hz="${hz}" h_fov="${h_fov}" width="1440" height="1080" format="${format}" frame_id="${namespace}/${name}_link"/>
     </xacro:macro>
 </robot>

File: urdf/gazebo/camera.gazebo.xacro (robot description, xacro)
@@ -2,5 +2,5 @@
 <robot xmlns:xacro="http://www.ros.org/wiki/xacro">
     <xacro:macro name="gazebo_camera" params="name reference hz h_fov width height format frame_id">
-    <gazebo reference="${reference}">
+    <gazebo reference="${namespace}/${reference}">
         <sensor type="camera" name="${name}_sensor">
             <update_rate>${hz}</update_rate>
@@ -28,8 +28,8 @@
                 <alwaysOn>true</alwaysOn>
                 <updateRate>${hz}</updateRate>
-                <cameraName>${name}</cameraName>
+                <cameraName>${namespace}/${name}</cameraName>
                 <imageTopicName>image_raw</imageTopicName>
                 <cameraInfoTopicName>camera_info</cameraInfoTopicName>
-                <frameName>${frame_id}</frameName>
+                <frameName>${namespace}/${frame_id}</frameName>
                 <autoDistortion>true</autoDistortion>
             </plugin>

File: urdf/gazebo/lidar.gazebo.xacro (robot description, xacro)
@@ -3,5 +3,5 @@
     <xacro:property name="use_gpu"  value="true"/>
     <xacro:macro name="gazebo_lidar" params="name topic_points hz lasers samples min_range max_range noise min_angle max_angle vfov_min vfov_max gpu">
-    <gazebo reference="${name}_link">
+    <gazebo reference="${namespace}/${name}_link">
         <xacro:if value="${gpu}">
             <sensor type="gpu_ray" name="${name}_sensor">
@@ -36,5 +36,5 @@
                 <max_range>${max_range}</max_range>
                 <gaussianNoise>${noise}</gaussianNoise>
-                <robotNamespace>/</robotNamespace>
+                <robotNamespace>/${namespace}</robotNamespace>
             </plugin>
             </sensor>
@@ -72,5 +72,5 @@
                 <max_range>${max_range}</max_range>
                 <gaussianNoise>${noise}</gaussianNoise>
-                <robotNamespace>/</robotNamespace>
+                <robotNamespace>/${namespace}</robotNamespace>
             </plugin>
             </sensor>

File: urdf/hesai/pandar_XT32.urdf.xacro (robot description, xacro)
@@ -3,11 +3,11 @@
     <xacro:include filename="$(find gazebo_sensor_collection)/urdf/gazebo/lidar.gazebo.xacro" />
     <xacro:property name="M_PI" value="3.1415926535897931" />
-    <xacro:macro name="pandar_XT32" params="*origin parent:=base_link name:=pandar topic_points:=/pandar/points gpu:=true">
+    <xacro:macro name="pandar_XT32" params="*origin parent:=base_link name:=pandar topic_points:=/points gpu:=true">
     <joint name="${name}_frame_joint" type="fixed">
         <xacro:insert_block name="origin" />
         <parent link="${parent}"/>
-        <child link="${name}_link"/>
+        <child link="${namespace}/${name}_link"/>
     </joint>
-    <link name="${name}_link">
+    <link name="${namespace}/${name}_link">
         <inertial>
             <mass value="0.455"/>
@@ -22,7 +22,8 @@
         </collision>
         <visual name="base_visual">
-            <origin xyz="0 0 0.0" rpy="0 0 0" />
+            <origin xyz="0 0 0.0" rpy="${M_PI/2} 0 ${M_PI}" />
             <geometry>
-                <cylinder radius="0.05" length="0.076"/>
+                <mesh filename="package://gazebo_sensor_collection/meshes/pandar/pandar_xt32.stl"
+                      scale="0.001 0.001 0.001"/>
             </geometry>
         </visual>

File: urdf/hesai/pandar_XT32M2X.urdf.xacro (robot description, xacro)
@@ -3,11 +3,11 @@
     <xacro:include filename="$(find gazebo_sensor_collection)/urdf/gazebo/lidar.gazebo.xacro" />
     <xacro:property name="M_PI" value="3.1415926535897931" />
-    <xacro:macro name="pandar_XT32M2X" params="*origin parent:=base_link name:=pandar topic_points:=/pandar/points hz:=10 gpu:=true">
+    <xacro:macro name="pandar_XT32M2X" params="*origin parent:=base_link name:=pandar topic_points:=/points hz:=10 gpu:=true">
     <joint name="${name}_frame_joint" type="fixed">
         <xacro:insert_block name="origin" />
         <parent link="${parent}"/>
-        <child link="${name}_link"/>
+        <child link="${namespace}/${name}_link"/>
     </joint>
-    <link name="${name}_link">
+    <link name="${namespace}/${name}_link">
         <inertial>
             <mass value="0.49"/>
@@ -22,7 +22,8 @@
         </collision>
         <visual name="base_visual">
-            <origin xyz="0 0 0.0" rpy="0 0 0" />
+            <origin xyz="0 0 0.0" rpy="${M_PI/2} 0 ${M_PI}" />
             <geometry>
-                <cylinder radius="0.05" length="0.076"/>
+                <mesh filename="package://gazebo_sensor_collection/meshes/pandar/pandar_xt32.stl"
+                      scale="0.001 0.001 0.001"/>
             </geometry>
         </visual>

File: urdf/ouster/OS0.urdf.xacro (robot description, xacro)
@@ -7,7 +7,7 @@
         <xacro:insert_block name="origin" />
         <parent link="${parent}"/>
-        <child link="${name}_link"/>
+        <child link="${namespace}/${name}_link"/>
     </joint>
-    <link name="${name}_link">
+    <link name="${namespace}/${name}_link">
         <inertial>
             <mass value="0.455"/>

File: urdf/ouster/OS1.urdf.xacro (robot description, xacro)
@@ -8,7 +8,7 @@
         <xacro:insert_block name="origin" />
         <parent link="${parent}"/>
-        <child link="${name}_link"/>
+        <child link="${namespace}/${name}_link"/>
     </joint>
-    <link name="${name}_link">
+    <link name="${namespace}/${name}_link">
         <inertial>
             <mass value="0.455"/>
