Commit message: added hesai, ouster, firefly and econ sensors

File: urdf/gazebo/lidar.gazebo.xacro (robot description, xacro)
@@ -2,5 +2,5 @@
 <robot xmlns:xacro="http://www.ros.org/wiki/xacro">
     <xacro:property name="use_gpu"  value="true"/>
-    <xacro:macro name="lidar_gazebo" params="name topic_points hz lasers samples min_range max_range noise min_angle max_angle vfov_min vfov_max gpu">
+    <xacro:macro name="gazebo_lidar" params="name topic_points hz lasers samples min_range max_range noise min_angle max_angle vfov_min vfov_max gpu">
     <gazebo reference="${name}_link">
         <xacro:if value="${gpu}">
@@ -31,9 +31,10 @@
             </ray>
             <plugin name="${name}_gazebo_ros_laser_controller" filename="libgazebo_ros_lidar_gpu.so">
-                <topicName>${topic_points}</topicName>
+                <topicName>/${namespace}/${topic_points}</topicName>
                 <frameName>${name}_link</frameName>
                 <min_range>${min_range}</min_range>
                 <max_range>${max_range}</max_range>
                 <gaussianNoise>${noise}</gaussianNoise>
+                <robotNamespace>/</robotNamespace>
             </plugin>
             </sensor>
@@ -66,9 +67,10 @@
             </ray>
             <plugin name="${name}_gazebo_ros_laser_controller" filename="libgazebo_ros_lidar.so">
-                <topicName>${topic_points}</topicName>
+                <topicName>/${namespace}/${topic_points}</topicName>
                 <frameName>${name}_link</frameName>
                 <min_range>${min_range}</min_range>
                 <max_range>${max_range}</max_range>
                 <gaussianNoise>${noise}</gaussianNoise>
+                <robotNamespace>/</robotNamespace>
             </plugin>
             </sensor>

File: urdf/hesai/pandar_XT32.urdf.xacro (robot description, xacro)
@@ -3,6 +3,5 @@
     <xacro:include filename="$(find gazebo_sensor_collection)/urdf/gazebo/lidar.gazebo.xacro" />
     <xacro:property name="M_PI" value="3.1415926535897931" />
-    <xacro:macro name="OS1" params="*origin parent:=base_link name:=os0 topic_points:=/os1/points hz:=10 lasers:=64 samples:=1024
-                                    noise:=0.01 gpu:=true">
+    <xacro:macro name="pandar_XT32" params="*origin parent:=base_link name:=pandar topic_points:=/pandar/points gpu:=true">
     <joint name="${name}_frame_joint" type="fixed">
         <xacro:insert_block name="origin" />
@@ -19,17 +18,17 @@
             <origin xyz="0 0 0" rpy="0 0 0" />
             <geometry>
-                <cylinder radius="0.04" length="0.073"/>
+                <cylinder radius="0.05" length="0.076"/>
             </geometry>
         </collision>
         <visual name="base_visual">
-            <origin xyz="0 0 0.0" rpy="0 0 1.5707" />
+            <origin xyz="0 0 0.0" rpy="0 0 0" />
             <geometry>
-                <mesh filename="package://gazebo_sensor_collection/meshes/ouster/ouster.dae" />
+                <cylinder radius="0.05" length="0.076"/>
             </geometry>
         </visual>
     </link>
-    <xacro:gazebo_lidar name="${name}" topic_points="${topic_points}" hz="${hz}" lasers="${lasers}" samples="${samples}"
-                      min_range="0.3" max_range="120" noise="${noise}" min_angle="-${M_PI}"
-                      max_angle="${M_PI}" vfov_min="-0.3927" vfov_max="0.3927" gpu="${gpu}"/>
+    <xacro:gazebo_lidar name="${name}" topic_points="${topic_points}" hz="10" lasers="32" samples="2000"
+                      min_range="0.1" max_range="120" noise="0.005" min_angle="-${M_PI}"
+                      max_angle="${M_PI}" vfov_min="-0.279253" vfov_max="0.261799" gpu="${gpu}"/>
     </xacro:macro>
 </robot>

Commit message: added xsens

File: urdf/gazebo/lidar.gazebo.xacro (robot description, xacro)
@@ -1,5 +1,4 @@
 <?xml version="1.0"?>
 <robot xmlns:xacro="http://www.ros.org/wiki/xacro">
-    <xacro:property name="use_gpu"  value="true"/>
     <xacro:macro name="gazebo_lidar" params="name topic_points hz lasers samples min_range max_range noise min_angle max_angle vfov_min vfov_max gpu">
     <gazebo reference="${namespace}/${name}_link">
